File: hw/whoop-v0.11td.sch (EAGLE design)
At the start: 70 parts, among them IC1 MCP1703CB, IC2 STM32F103CBT6, Q1 AO3401, Q2 SI2312, Q3 SI2312, Q4 SI2312, Q5 SI2312, Q6 2N7002, U1 A7105, X1 BAT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

Commit message: hw update
Parts:
- C23: value 2u2 -> 4u7
- C4: value u47 -> 4u7
- IC3: value MPU-9250 -> MPU6500
- renumbered U$1 to IC3, U1 to IC4
Connections:
- removed net FLEXI_RX/SDA: IC2.PB11
- removed net FLEXI_TX/SCL: IC2.PB10
- removed net MAIN_RX: IC2.PA10
- removed net MAIN_TX: IC2.PA9
Other:
- moved on the sheet: J1, L1, PAD1, R3
