File: hw/v.2/whoop-v2.0-F3.brd (EAGLE design)
At the start: 11.7 x 36.3 mm, 73 parts, among them IC1 MCP1703T-3002E/CB, IC2 MPU6500, IC3 STM32F303CCT6, IC4 A7105-1, Q1 AO3401, Q2 SI2312, Q3 SI2312, Q4 SI2312, Q5 SI2312, X1 M1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

Commit message: edit some values
Parts:
- C24: value 33p -> 27p
- R1: value 2k2 -> 5k1
Changed lines of the file:
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@@
 </element>
 <element name="C2" library="RC.v2" package="0402" value="0u1" x="-1.651" y="17.907" smashed="yes">
-<attribute name="NAME" x="-1.016" y="18.7706" size="0.3048" layer="25" font="vector" align="bottom-center"/>
-<attribute name="VALUE" x="-0.889" y="18.3134" size="0.3048" layer="27" font="vector" rot="R180" align="top-center"/>
+<attribute name="NAME" x="-1.651" y="18.7706" size="0.3048" layer="25" font="vector" align="bottom-center"/>
+<attribute name="VALUE" x="-1.651" y="18.3134" size="0.3048" layer="27" font="vector" rot="R180" align="top-center"/>
 </element>
 <element name="Q1" library="cc3d" package="SOT-23" value="AO3401" x="0.889" y="24.257" smashed="yes" rot="R180">
@@
 </element>
 <element name="C1" library="RC.v2" package="0402" value="10n" x="-0.0508" y="17.907" smashed="yes" rot="R180">
-<attribute name="NAME" x="0.508" y="18.7706" size="0.3048" layer="25" font="vector" align="bottom-center"/>
-<attribute name="VALUE" x="0.3556" y="18.3134" size="0.3048" layer="27" font="vector" rot="R180" align="top-center"/>
+<attribute name="NAME" x="0" y="18.7706" size="0.3048" layer="25" font="vector" align="bottom-center"/>
+<attribute name="VALUE" x="-0.0254" y="18.3134" size="0.3048" layer="27" font="vector" rot="R180" align="top-center"/>
 </element>
 <element name="C27" library="RC.v2" package="0402" value="1u" x="-2.1082" y="10.1092" smashed="yes" rot="R180">
@@
 <attribute name="VALUE" x="-3.2258" y="9.7282" size="0.3048" layer="27" font="vector" rot="R180" align="top-center"/>
 </element>
-<element name="R1" library="RC.v2" package="0402" value="2k2" x="3.81" y="10.8712" smashed="yes">
+<element name="R1" library="RC.v2" package="0402" value="5k1" x="3.81" y="10.8712" smashed="yes">
 <attribute name="NAME" x="4.8768" y="11.049" size="0.3048" layer="25" font="vector" align="bottom-center"/>
 <attribute name="VALUE" x="5.0038" y="10.6172" size="0.3048" layer="27" font="vector" rot="R180" align="top-center"/>
@@
 <attribute name="VALUE" x="5.334" y="4.318" size="0.3048" layer="27" font="vector" rot="R180" align="top-center"/>
 </element>
-<element name="C24" library="RC.v2" package="0402" value="33p" x="3.937" y="9.271" smashed="yes" rot="R180">
+<element name="C24" library="RC.v2" package="0402" value="27p" x="3.937" y="9.271" smashed="yes" rot="R180">
 <attribute name="NAME" x="5.1562" y="9.4488" size="0.3048" layer="25" font="vector" align="bottom-center"/>
 <attribute name="VALUE" x="5.1308" y="9.017" size="0.3048" layer="27" font="vector" rot="R180" align="top-center"/>
