File: hw/v.2/whoop-v2.0-F3.sch (EAGLE design)
At the start: 73 parts, among them IC1 MCP1703T-3002E/CB, IC2 MPU6500, IC3 STM32F303CCT6, IC4 A7105-1, Q1 AO3401, Q2 SI2312, Q3 SI2312, Q4 SI2312, Q5 SI2312, X1 M1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

Commit message: edit some values
Parts:
- C24: value 33p -> 27p
- R1: value 2k2 -> 5k1
Changed lines of the file:
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@@
 <setting verticaltext="up"/>
 </settings>
-<grid distance="0.05" unitdist="inch" unit="inch" style="lines" multiple="1" display="no" altdistance="0.01" altunitdist="inch" altunit="inch"/>
+<grid distance="0.1" unitdist="inch" unit="inch" style="lines" multiple="1" display="no" altdistance="0.01" altunitdist="inch" altunit="inch"/>
 <layers>
 <layer number="1" name="Top" color="4" fill="1" visible="no" active="no"/>
@@
 <part name="GND4" library="supply1" deviceset="GND" device=""/>
 <part name="C27" library="RC.v2" deviceset="C" device="0402" value="1u"/>
-<part name="R1" library="RC.v2" deviceset="R" device="0402" value="2k2"/>
+<part name="R1" library="RC.v2" deviceset="R" device="0402" value="5k1"/>
 <part name="R2" library="RC.v2" deviceset="R" device="0402" value="1k"/>
 <part name="C3" library="RC.v2" deviceset="C" device="0402" value="10n"/>
@@
 <part name="Y2" library="thermo" deviceset="FA-" device="3225" value="16 MHz"/>
 <part name="C23" library="RC.v2" deviceset="C" device="0402" value="33p"/>
-<part name="C24" library="RC.v2" deviceset="C" device="0402" value="33p"/>
+<part name="C24" library="RC.v2" deviceset="C" device="0402" value="27p"/>
 <part name="GND16" library="supply1" deviceset="GND" device=""/>
 <part name="C16" library="RC.v2" deviceset="C" device="0402" value="120p"/>
